File: frankenstein_lightningbolt.kicad_pcb (KiCad board)
At the start: 4 copper layers, 0 parts

Commit message: Routing v1
Parts:
- added C1: 22uF 25V 1206 RoHS, easyeda2kicad:C1206, F.Cu at (94.5, 59.9)
- added C2: 22uF 25V 1206 RoHS, easyeda2kicad:C1206, F.Cu at (103.6, 59.9)
- added C3: 1uF 50V 1206 RoHS, easyeda2kicad:C1206, F.Cu at (79.8, 76.2)
- added C4: 1uF 50V 1206 RoHS, easyeda2kicad:C1206, F.Cu at (79.8, 73.7)
- added C5: 100nF 50V 1206 RoHS, easyeda2kicad:C1206, F.Cu at (79.8, 71.1)
- added C6: 1uF 50V 1206 RoHS, easyeda2kicad:C1206, F.Cu at (71.6, 76.2)
- added D1: SMF05CT1G, easyeda2kicad:SOT-363_L2.0-W1.3-P0.65-LS2.1-BR, F.Cu at (110.5, 66.5)
- added J1: 12V OUT, Connector_PinHeader_2.54mm:PinHeader_1x02_P2.54mm_Vertical, F.Cu at (106.7, 57.9)
- added J2: 3V3 OUT, Connector_PinHeader_2.54mm:PinHeader_1x02_P2.54mm_Vertical, F.Cu at (97.8, 57.9)
- added J3: 5V OUT, Connector_PinHeader_2.54mm:PinHeader_1x02_P2.54mm_Vertical, F.Cu at (88.4, 57.9)
- added Q1: DMP3013SFV-7, easyeda2kicad:POWERPAK-1212-8_L3.1-W3.1-P0.65-LS3.3-BL, F.Cu at (86.6, 74.9)
- added Q2: DMP3013SFV-7, easyeda2kicad:POWERPAK-1212-8_L3.1-W3.1-P0.65-LS3.3-BL, F.Cu at (93.0, 74.9)
- added R1: 1KOhms ±1% 1/4W 1206 RoHS, easyeda2kicad:R1206, F.Cu at (99.1, 72.9)
- added R2: 10KOhms 1206, easyeda2kicad:R1206, F.Cu at (99.1, 75.4)
- added R3: 47KOhms ±1% 1/8W 0805 RoHS, easyeda2kicad:R0805, F.Cu at (90.4, 71.6)
- added R4: 5.1k 0603, easyeda2kicad:R0603, F.Cu at (83.8, 58.2)
- added R5: 2.4k 0603, easyeda2kicad:R0603, F.Cu at (79.0, 58.2)
- added R6: 5.1k 0603, easyeda2kicad:R0603, F.Cu at (83.8, 56.6)
- added R7: 2.4k 0603, easyeda2kicad:R0603, F.Cu at (79.0, 56.6)
- added R8: 5.1k 0603, easyeda2kicad:R0603, F.Cu at (83.8, 59.7)
- added R9: 10k 0603, easyeda2kicad:R0603, F.Cu at (79.0, 59.7)
- added REF**: frankenlogo, frankenlogo:frankenlogo, B.Cu at (108.7, 73.0)
- added U1: CYPD3177-24LQXQ, easyeda2kicad:TQFN-24_L4.0-W4.0-P0.50-TL-EP2.8, F.Cu at (81.0, 66.0)
- added U2: AMS1117-3.3, easyeda2kicad:SOT-223-3_L6.5-W3.4-P2.30-LS7.0-BR, F.Cu at (100.3, 64.5)
- added U3: AMS1117-5.0, easyeda2kicad:SOT-223_L6.5-W3.5-P2.30-LS7.0-BR, F.Cu at (90.9, 64.5)
- added USB1: AF10.0 Aparagraph After the two feet Boundless iron LCP Vin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, easyeda2kicad:USB-A-SMD_JTJ-USB-AF-10.0-023, F.Cu at (117.5, 66.6)
- added USBC1: USB3.1C16PFSMT, easyeda2kicad:USB-C-SMD_TYPE-C-USB-17, F.Cu at (71.1, 66.5)
Routing:
- net /USB+: track 0.00 -> 83.1 mm, vias 0 -> 2
- net /USB-: track 0.00 -> 70.4 mm, vias 0 -> 2
- net GND: track 0.00 -> 51.4 mm, vias 0 -> 23
- net +5V: track 0.00 -> 43.6 mm, vias 0 -> 1
- net /VBUS_FET_EN: track 0.00 -> 43.1 mm, vias 0 -> 5
- net /VDDD: track 0.00 -> 32.2 mm
- net VBUS: track 0.00 -> 25.0 mm, vias 0 -> 8
- net /VBUS_MIN: track 0.00 -> 19.0 mm, vias 0 -> 2
- net Net-(U1-VBUS_FET_EN): track 0.00 -> 18.3 mm, vias 0 -> 2
- net /VBUS_MAX: track 0.00 -> 17.6 mm, vias 0 -> 2
- net Vdrive: track 0.00 -> 14.4 mm, vias 0 -> 10
- net /ISNK_COARSE: track 0.00 -> 14.2 mm
- net +3V3: track 0.00 -> 12.9 mm
- net Net-(Q1-S-Pad1): track 0.00 -> 12.3 mm
- net Net-(U1-VCCD): track 0.00 -> 9.43 mm, vias 0 -> 2
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- added copper zone on In2.Cu, net GND
- added copper zone on In1.Cu, net VBUS
- added copper zone on In1.Cu, net Vdrive
Other:
- board outline added: 61.5 x 22.9 mm
- board text added: "12V GND"
- board text added: "3V3 GND"
- board text added: "5V GND"
- board text added: "Frankenstein Lightning Bolt USB-C Passthrough with Power Breakout 3.3V 5V 12V (C) wirkbetrieb.net / Tom Merlin Eichhorn"
